File: Micromouse_Board/micro_schematic.sch (EAGLE design)
At the start: 44 parts, among them IC1 L293B, IC2 DSPIC33FJ64MC804-X_PT, J1 61300211121, J2 61300611121, J3 61300311121, J4 61300311121, J5 61300311121, J6 61300611121, U1 TPS62163, U2 Value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

Commit message: Updated board version
Parts:
- added LED3: HSME-C170, SamacSys_Parts:HSME-C170
- added LED4: SSL-LX5093TC, SSL-LX5093TC:SSL-LX5093TC
- added R4: 4k7, rcl:R-US_R0805
- added R5, R7: 1k, rcl:R-US_R0805
- added R6: 180, rcl:R-US_R0805
- added S2: PTS647SM50SMTR2LFS, SamacSys_Parts:PTS647SM50SMTR2LFS
- added T1: (no value), zetex:NMOSSOT23
- C5, C6: value 120pF -> 22pF
- U1: value TPS62163 -> Value
Connections:
- net N$11 renamed P43
- net N$29 renamed P24
- removed net N$10: IC2.PGEC3/ASCL1/RP6/CN24/PMD6/RB6, JP3.13
- removed net N$12: IC2.RP21/CN26/PMA3/RC5, JP3.16
- removed net N$13: IC2.RP20/CN25/PMA4/RC4, JP3.14
- removed net N$14: IC2.RP19/CN28/PMBE/RC3, JP3.12
- removed net N$15: IC2.TDI/PMA9/RA9, JP3.9
- removed net N$16: IC2.SOSCO/T1CK/CN0/RA4, JP3.10
- removed net N$17: IC2.SOSCI/RP4/CN1/RB4, JP3.8
- removed net N$18: IC2.TDO/PMA8/RA8, JP3.6
- removed net N$19: IC2.PWM2H1/RP22/CN18/PMA1/RC6, JP3.7
- removed net N$20: IC2.PWM2L1/RP23/CN17/PMA0/RC7, JP3.5
- removed net N$23: IC2.PWM1H2/DAC1RP/RP12/CN14/PMD0/RB12, JP3.3
- removed net N$30: IC2.AN6/DAC1RM/RP16/CN8/RC0, JP3.2
- removed net N$9: IC2.PGED3/ASDA1/RP5/CN27/PMD7/RB5, JP3.15
- new net BUTTON1: IC2.PWM1H1/DAC1LP/RTCC/RP14/CN12/PMWR/RB14, R4.2, S2.3, S2.4
- new net LED3: IC2.PWM1H2/DAC1RP/RP12/CN14/PMD0/RB12, R5.2
- new net LED4: IC2.TDO/PMA8/RA8, JP3.2, R7.1
- new net N$21: LED4.A, R7.2
- new net N$6: R5.1, T1.G
- new net N$8: LED3.A, R6.2
- new net P11: IC2.PWM1L2/DAC1RN/RP13/CN13/PMRD/RB13, JP3.14
- new net P2: IC2.PWM2H1/RP22/CN18/PMA1/RC6, JP3.13
- new net P25: IC2.AN6/DAC1RM/RP16/CN8/RC0, JP3.4
- new net P33: IC2.SOSCI/RP4/CN1/RB4, JP3.3
- new net P34: IC2.SOSCO/T1CK/CN0/RA4, JP3.6
- new net P35: IC2.TDI/PMA9/RA9, JP3.5
- new net P36: IC2.RP19/CN28/PMBE/RC3, JP3.8
- new net P37: IC2.RP20/CN25/PMA4/RC4, JP3.7
- new net P38: IC2.RP21/CN26/PMA3/RC5, JP3.10
- new net P41: IC2.PGED3/ASDA1/RP5/CN27/PMD7/RB5, JP3.9
- new net P42: IC2.PGEC3/ASCL1/RP6/CN24/PMD6/RB6, JP3.12
- net +3V3: now also JP3.15, S2.1, S2.2
- net +5V: now also R6.1
- net GND: now also JP3.16, LED4.K, R4.1, T1.S
- net M1_1: now also D4.K, D5.A; no longer D2.K, D3.A
- net M1_2: now also D2.K, D3.A; no longer D4.K, D5.A
- net M2_1: now also D8.K, D9.A; no longer D6.K, D7.A
- net M2_2: now also D6.K, D7.A; no longer D8.K, D9.A
- net N$22: now also LED3.K, T1.D; no longer IC2.PWM1H1/DAC1LP/RTCC/RP14/CN12/PMWR/RB14, JP3.4
- net PWM2: now also IC2.PWM2L1/RP23/CN17/PMA0/RC7; no longer IC2.PWM1L2/DAC1RN/RP13/CN13/PMRD/RB13
